Commit message: Add pid parameters for simulation. Update dynamics.

File: robotiq_description/urdf/robotiq_gripper_macro.urdf.xacro (robot description, xacro)
@@ -166,12 +166,14 @@
             <origin xyz="0.03060114 0.0 0.05490452" rpy="0 0 0" />
             <limit lower="0.0" upper="0.8" velocity="0.5" effort="50" />
-        </joint>
-        <joint name="${prefix}robotiq_85_right_knuckle_joint" type="revolute">
+            <dynamics damping="0.5"/>
+        </joint>
+        <joint name="${prefix}robotiq_85_right_knuckle_joint" type="continuous">
             <parent link="${prefix}robotiq_85_base_link" />
             <child link="${prefix}robotiq_85_right_knuckle_link" />
             <axis xyz="0 -1 0" />
             <origin xyz="-0.03060114 0.0 0.05490452" rpy="0 0 0" />
-            <limit lower="-0.8" upper="0.0" velocity="0.5" effort="50" />
             <mimic joint="${prefix}robotiq_85_left_knuckle_joint" multiplier="-1" />
+<!--            <dynamics damping="1.0" friction="0.1"/>-->
+            <limit lower="-0.8" upper="0.8" velocity="0.5" effort="50" />
         </joint>
         <joint name="${prefix}robotiq_85_left_finger_joint" type="fixed">
@@ -185,5 +187,5 @@
             <origin xyz="-0.03152616 0.0 -0.00376347" rpy="0 0 0" />
         </joint>
-        <joint name="${prefix}robotiq_85_left_inner_knuckle_joint" type="continuous">
+        <joint name="${prefix}robotiq_85_left_inner_knuckle_joint" type="revolute">
             <parent link="${prefix}robotiq_85_base_link" />
             <child link="${prefix}robotiq_85_left_inner_knuckle_link" />
@@ -191,4 +193,6 @@
             <origin xyz="0.0127 0.0 0.06142" rpy="0 0 0" />
             <mimic joint="${prefix}robotiq_85_left_knuckle_joint" />
+            <dynamics damping="0.5"/>
+            <limit lower="-0.8" upper="0.8" velocity="0.5" effort="50" />
         </joint>
         <joint name="${prefix}robotiq_85_right_inner_knuckle_joint" type="continuous">
@@ -198,6 +202,8 @@
             <origin xyz="-0.0127 0.0 0.06142" rpy="0 0 0" />
             <mimic joint="${prefix}robotiq_85_left_knuckle_joint" multiplier="-1" />
-        </joint>
-        <joint name="${prefix}robotiq_85_left_finger_tip_joint" type="continuous">
+<!--            <dynamics damping="1.0" friction="0.1"/>-->
+            <limit lower="-0.8" upper="0.8" velocity="0.5" effort="50" />
+        </joint>
+        <joint name="${prefix}robotiq_85_left_finger_tip_joint" type="revolute">
             <parent link="${prefix}robotiq_85_left_finger_link" />
             <child link="${prefix}robotiq_85_left_finger_tip_link" />
@@ -205,4 +211,6 @@
             <origin xyz="0.00563134 0.0 0.04718515" rpy="0 0 0" />
             <mimic joint="${prefix}robotiq_85_left_knuckle_joint" multiplier="-1" />
+            <dynamics damping="0.5"/>
+            <limit lower="-0.8" upper="0.8" velocity="0.5" effort="50" />
         </joint>
         <joint name="${prefix}robotiq_85_right_finger_tip_joint" type="continuous">
@@ -212,4 +220,6 @@
             <origin xyz="-0.00563134 0.0 0.04718515" rpy="0 0 0" />
             <mimic joint="${prefix}robotiq_85_left_knuckle_joint" />
+<!--            <dynamics damping="0.5"/>-->
+            <limit lower="-0.8" upper="0.8" velocity="0.5" effort="50" />
         </joint>
     </xacro:macro>

File: robotiq_description/urdf/robotiq_sim_gripper.ros2_control.xacro (robot description, xacro)
@@ -27,4 +27,20 @@
                         <param name="initial_value">0.2</param>
                     </state_interface>
+                    <param name="p_pos">25.0</param>
+                    <param name="i_pos">0.0</param>
+                    <param name="d_pos">0.25</param>
+                    <param name="iMax_pos">1.0</param>
+                    <param name="iMin_pos">-1.0</param>
+                    <param name="cmdMax_pos">2.0</param>
+                    <param name="cmdMin_pos">-2.0</param>
+                    <param name="cmdOffset_pos">0.0</param>
+                    <param name="p_vel">0.25</param>
+                    <param name="i_vel">0.025</param>
+                    <param name="d_vel">0.0</param>
+                    <param name="iMax_vel">25.0</param>
+                    <param name="iMin_vel">-25.0</param>
+                    <param name="cmdMax_vel">1000.0</param>
+                    <param name="cmdMin_vel">-1000.0</param>
+                    <param name="cmdOffset_vel">0.0</param>
                 </xacro:if>
                 <xacro:unless value="${sim_ignition}">
@@ -43,4 +59,22 @@
                     <state_interface name="velocity"/>
                 </xacro:unless>
+                <xacro:if value="${sim_ignition}">
+                    <param name="p_pos">10.0</param>
+                    <param name="i_pos">0.0</param>
+                    <param name="d_pos">0.0</param>
+                    <param name="iMax_pos">1.0</param>
+                    <param name="iMin_pos">-1.0</param>
+                    <param name="cmdMax_pos">2.0</param>
+                    <param name="cmdMin_pos">-2.0</param>
+                    <param name="cmdOffset_pos">0.0</param>
+                    <param name="p_vel">0.1</param>
+                    <param name="i_vel">0.001</param>
+                    <param name="d_vel">0.0</param>
+                    <param name="iMax_vel">25.0</param>
+                    <param name="iMin_vel">-25.0</param>
+                    <param name="cmdMax_vel">50.0</param>
+                    <param name="cmdMin_vel">-50.0</param>
+                    <param name="cmdOffset_vel">0.0</param>
+                </xacro:if>
             </joint>
             <joint name="robotiq_85_left_inner_knuckle_joint">
@@ -52,4 +86,22 @@
                     <state_interface name="velocity"/>
                 </xacro:unless>
+                <xacro:if value="${sim_ignition}">
+                    <param name="p_pos">10.0</param>
+                    <param name="i_pos">0.0</param>
+                    <param name="d_pos">0.0</param>
+                    <param name="iMax_pos">1.0</param>
+                    <param name="iMin_pos">-1.0</param>
+                    <param name="cmdMax_pos">2.0</param>
+                    <param name="cmdMin_pos">-2.0</param>
+                    <param name="cmdOffset_pos">0.0</param>
+                    <param name="p_vel">0.1</param>
+                    <param name="i_vel">0.001</param>
+                    <param name="d_vel">0.0</param>
+                    <param name="iMax_vel">25.0</param>
+                    <param name="iMin_vel">-25.0</param>
+                    <param name="cmdMax_vel">50.0</param>
+                    <param name="cmdMin_vel">-50.0</param>
+                    <param name="cmdOffset_vel">0.0</param>
+                </xacro:if>
             </joint>
             <joint name="robotiq_85_right_inner_knuckle_joint">
@@ -61,4 +113,22 @@
                     <state_interface name="velocity"/>
                 </xacro:unless>
+                <xacro:if value="${sim_ignition}">
+                    <param name="p_pos">10.0</param>
+                    <param name="i_pos">0.0</param>
+                    <param name="d_pos">0.0</param>
+                    <param name="iMax_pos">1.0</param>
+                    <param name="iMin_pos">-1.0</param>
+                    <param name="cmdMax_pos">2.0</param>
+                    <param name="cmdMin_pos">-2.0</param>
+                    <param name="cmdOffset_pos">0.0</param>
+                    <param name="p_vel">0.1</param>
+                    <param name="i_vel">0.001</param>
+                    <param name="d_vel">0.0</param>
+                    <param name="iMax_vel">25.0</param>
+                    <param name="iMin_vel">-25.0</param>
+                    <param name="cmdMax_vel">50.0</param>
+                    <param name="cmdMin_vel">-50.0</param>
+                    <param name="cmdOffset_vel">0.0</param>
+                </xacro:if>
             </joint>
             <joint name="robotiq_85_left_finger_tip_joint">
@@ -70,4 +140,22 @@
                     <state_interface name="velocity"/>
                 </xacro:unless>
+                <xacro:if value="${sim_ignition}">
+                    <param name="p_pos">10.0</param>
+                    <param name="i_pos">0.0</param>
+                    <param name="d_pos">0.0</param>
+                    <param name="iMax_pos">1.0</param>
+                    <param name="iMin_pos">-1.0</param>
+                    <param name="cmdMax_pos">2.0</param>
+                    <param name="cmdMin_pos">-2.0</param>
+                    <param name="cmdOffset_pos">0.0</param>
+                    <param name="p_vel">0.1</param>
+                    <param name="i_vel">0.001</param>
+                    <param name="d_vel">0.0</param>
+                    <param name="iMax_vel">25.0</param>
+                    <param name="iMin_vel">-25.0</param>
+                    <param name="cmdMax_vel">50.0</param>
+                    <param name="cmdMin_vel">-50.0</param>
+                    <param name="cmdOffset_vel">0.0</param>
+                </xacro:if>
             </joint>
             <joint name="robotiq_85_right_finger_tip_joint">
@@ -79,4 +167,22 @@
                     <state_interface name="velocity"/>
                 </xacro:unless>
+                <xacro:if value="${sim_ignition}">
+                    <param name="p_pos">10.0</param>
+                    <param name="i_pos">0.0</param>
+                    <param name="d_pos">0.0</param>
+                    <param name="iMax_pos">1.0</param>
+                    <param name="iMin_pos">-1.0</param>
+                    <param name="cmdMax_pos">2.0</param>
+                    <param name="cmdMin_pos">-2.0</param>
+                    <param name="cmdOffset_pos">0.0</param>
+                    <param name="p_vel">0.1</param>
+                    <param name="i_vel">0.001</param>
+                    <param name="d_vel">0.0</param>
+                    <param name="iMax_vel">25.0</param>
+                    <param name="iMin_vel">-25.0</param>
+                    <param name="cmdMax_vel">50.0</param>
+                    <param name="cmdMin_vel">-50.0</param>
+                    <param name="cmdOffset_vel">0.0</param>
+                </xacro:if>
             </joint>
             <!-- Only add this with fake hardware mode -->
